Commit message: Added Lidar cone detection and clustering

File: falcon_ws/src/eufs_sim/eufs_racecar/robots/eufs/robot.urdf.xacro (robot description, xacro)
@@ -51,5 +51,5 @@
     </xacro:VLP-16R> -->
     <xacro:rplidar_a1 parent="chassis" name="rplidar" topic="/gazebo_scan" hz="10" samples="720" active="$(arg simulate_perception)">
-        <origin xyz="1.543 0.0 0.36" rpy="0 0 0"/>
+        <origin xyz="1.683 0.0 0" rpy="0 0 0"/>
     </xacro:rplidar_a1>
     <xacro:zed_camera parent="chassis" prefix="zed" active="$(arg simulate_perception)">

File: falcon_ws/src/eufs_sim/eufs_sensors/urdf/lidar.urdf.xacro (robot description, xacro)
@@ -42,20 +42,19 @@
       <gazebo reference="${name}_link">
         <sensor type="ray" name="${name}_sensor">
-          <!-- RPLIDAR A1 specs -->
-          <update_rate>5.5</update_rate>      <!-- 5.5 Hz scan rate -->
-          <always_on>true</always_on>
+          <pose>0 0 0 0 0 0</pose>
           <visualize>true</visualize>
+          <update_rate>5.5</update_rate> <!-- 5.5 Hz Typical -->
           <ray>
             <scan>
               <horizontal>
-                <samples>360</samples>         <!-- 360 samples → ~1° resolution -->
+                <samples>1200</samples> <!-- 8000hz/5.5hz / (~360pts) -->
                 <resolution>1</resolution>
-                <min_angle>0</min_angle>       <!-- Full 360° scan -->
-                <max_angle>6.28318</max_angle>
+                <min_angle>-3.14159265</min_angle>
+                <max_angle>3.14159265</max_angle>
               </horizontal>
             </scan>
             <range>
-              <min>0.15</min>                <!-- Minimum distance -->
-              <max>6.0</max>                 <!-- Maximum distance -->
+              <min>0.15</min> <!-- 0.15m -->
+              <max>8.0</max> <!-- 12m -->
               <resolution>0.01</resolution>
             </range>
@@ -63,5 +62,5 @@
               <type>gaussian</type>
               <mean>0.0</mean>
-              <stddev>0.01</stddev>
+              <stddev>0.01</stddev> <!-- Typical noise level -->
             </noise>
           </ray>
@@ -69,6 +68,7 @@
                   filename="libgazebo_ros_ray_sensor.so">
             <ros>
-              <remapping>~/out:=${topic}</remapping>
+              <remapping>~/out:=/gazebo_scan</remapping>
             </ros>
+            <output_type>sensor_msgs/LaserScan</output_type>
             <frame_name>${name}_link</frame_name>
           </plugin>
