Commit message: added dependecies, foxglove bridge build and easy setting ups to setup_falcon.sh. Modified bringup launches with planning and mapping stacks with pseudo cones

File: falcon_ws/src/eufs_sim/eufs_racecar/urdf/wheels.urdf.xacro (robot description, xacro)
@@ -1,4 +1,7 @@
 <?xml version="1.0"?>
 <robot name="wheels" xmlns:xacro="http://www.ros.org/wiki/xacro">
+  <material name="tire_mat">
+    <color rgba="0.12 0.12 0.12 1.0"/>
+  </material>
   <xacro:macro name="wheels"
                params="chassis_width wheelbase">
