Commit message: Made changes to the URDF files

File: falcon_ws/src/eufs_sim/eufs_racecar/robots/ads-dv/robot.urdf.xacro (robot description, xacro)
@@ -51,5 +51,5 @@
     </xacro:VLP-16R> -->
     <xacro:rplidar_a1 parent="chassis" name="rplidar" topic="/gazebo_scan" hz="10" samples="720" active="$(arg simulate_perception)">
-        <origin xyz="0.443 0.0 0.3" rpy="0 ${6.1*M_PI/180.0} 0"/>
+        <origin xyz="0.443 0.0 0.3" rpy="0 0 0"/>
     </xacro:rplidar_a1>
     <xacro:zed_camera parent="chassis" prefix="zed" active="$(arg simulate_perception)">

File: falcon_ws/src/eufs_sim/eufs_racecar/robots/eufs/robot.urdf.xacro (robot description, xacro)
@@ -51,5 +51,5 @@
     </xacro:VLP-16R> -->
     <xacro:rplidar_a1 parent="chassis" name="rplidar" topic="/gazebo_scan" hz="10" samples="720" active="$(arg simulate_perception)">
-        <origin xyz="1.543 0.0 0.36" rpy="0 ${6.1*M_PI/180.0} 0"/>
+        <origin xyz="1.543 0.0 0.36" rpy="0 0 0"/>
     </xacro:rplidar_a1>
     <xacro:zed_camera parent="chassis" prefix="zed" active="$(arg simulate_perception)">

Commit message: added camera view to the teleop node

File: falcon_ws/src/eufs_sim/eufs_racecar/robots/ads-dv/robot.urdf.xacro (robot description, xacro)
@@ -56,4 +56,8 @@
 	    <origin xyz="0.334 0.0 0.295" rpy="0 ${10.15*M_PI/180.0} 0"/>
     </xacro:zed_camera>
+    <!-- Always-on teleop camera for falcon_teleop (no visual mesh, works in any launch_group) -->
+    <xacro:teleop_camera parent="chassis" prefix="teleop_camera">
+      <origin xyz="0.334 0.0 0.295" rpy="0 ${10.15*M_PI/180.0} 0"/>
+    </xacro:teleop_camera>
     <xacro:sensor_imu parent="chassis" prefix="zed_imu" topic_prefix="/camera">
         <origin xyz="0.334 0.0 0.295" rpy="0 ${10.15*M_PI/180.0} 0"/>

File: falcon_ws/src/eufs_sim/eufs_sensors/urdf/all_sensors.urdf.xacro (robot description, xacro)
@@ -13,3 +13,5 @@
   <!-- ZED Stereo camera -->
   <xacro:include filename="$(find eufs_sensors)/urdf/zed.urdf.xacro"/>
+  <!-- Teleop camera - always on, no visual, for falcon_teleop view in any launch_group -->
+  <xacro:include filename="$(find eufs_sensors)/urdf/teleop_camera.urdf.xacro"/>
 </robot>

Commit message: before getting rid of duplicate cone_fusion pipelines

File: falcon_ws/src/eufs_sim/eufs_racecar/robots/ads-dv/robot.urdf.xacro (robot description, xacro)
@@ -51,5 +51,5 @@
     </xacro:VLP-16R> -->
     <xacro:rplidar_a1 parent="chassis" name="rplidar" topic="/gazebo_scan" hz="10" samples="720" active="$(arg simulate_perception)">
-        <origin xyz="0.443 0.0 0.3" rpy="0 0 0"/>
+        <origin xyz="1.4 0.0 0" rpy="0 0 0"/>
     </xacro:rplidar_a1>
     <xacro:zed_camera parent="chassis" prefix="zed" active="$(arg simulate_perception)">

File: falcon_ws/src/eufs_sim/eufs_sensors/urdf/lidar.urdf.xacro (robot description, xacro)
@@ -50,6 +50,6 @@
                 <samples>1200</samples> <!-- 8000hz/5.5hz / (~360pts) -->
                 <resolution>1</resolution>
-                <min_angle>-3.14159265</min_angle>
-                <max_angle>3.14159265</max_angle>
+                <min_angle>-2.51327</min_angle>
+                <max_angle>2.51327</max_angle>
               </horizontal>
             </scan>
